Commit message: turret_controls
allow turret to be controlled by Control msg

File: src/sim_node/sim_node/models/hero/hero-blue.urdf (robot description, URDF)
Before this commit: robot hero, 6 links, 5 joints
Joints:
- joint turret_joint: axis 1 0 0 -> -1 0 0

File: src/sim_node/sim_node/models/hero/hero-red.urdf (robot description, URDF)
Before this commit: robot hero, 6 links, 5 joints
Joints:
- joint turret_joint: axis 1 0 0 -> -1 0 0

File: src/sim_node/sim_node/models/infantry/infantry-blue.urdf (robot description, URDF)
Before this commit: robot infantry, 6 links, 5 joints
Joints:
- joint turret_joint: axis 1 0 0 -> -1 0 0

File: src/sim_node/sim_node/models/infantry/infantry-red.urdf (robot description, URDF)
Before this commit: robot infantry, 6 links, 5 joints
Joints:
- joint turret_joint: axis 1 0 0 -> -1 0 0
